File: washing-machine-delayed-start/eagle/prototype-mark-II.brd (EAGLE design)
At the start: 100 x 80 mm, 19 parts

Commit message: Routes improvement
Parts:
- removed 6V: BATTERY_CONNDEANS, SparkFun-Connectors:DEANS
- added +: (no value), SparkFun-Connectors:JST-2-PTH-VERT
- moved R6 68.3 mm to (53.3, 25.4), turned to 180 degrees
- moved R5 53.2 mm to (49.5, 43.2), turned to 270 degrees
- moved R4 42.1 mm to (57.1, 45.7), turned to 270 degrees
- moved LED5 38.4 mm to (48.3, 52.1)
- moved SET_BTN 38.4 mm to (40.6, 25.4)
- moved R2 36.4 mm to (61.0, 33.0), turned to 270 degrees
- moved R3 35.2 mm to (62.2, 45.7), turned to 270 degrees
- moved VALID_BTN 33.7 mm to (40.6, 38.1)
- moved R7 33.0 mm to (40.6, 47.0), turned to 180 degrees
- moved R1 29.8 mm to (71.1, 35.6), turned to 180 degrees
- moved LED4 29.6 mm to (54.6, 52.1)
- moved LED1 28.0 mm to (73.7, 52.1)
- moved LED3 22.9 mm to (61.0, 52.1)
- moved LED2 22.2 mm to (67.3, 52.1)
- moved SW1 18.1 mm to (82.5, 21.6), turned to 90 degrees
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Connections:
- net GND: now also +.1; no longer 6V.-
- net N$16: now also +.2; no longer 6V.+
Routing:
- net GND: track 162.8 -> 93.6 mm
- net N$13: track 124.9 -> 75.1 mm
- net N$2: track 44.2 -> 16.6 mm
- net N$4: track 42.7 -> 18.4 mm
- net N$8: track 25.6 -> 2.58 mm
- net N$11: track 29.3 -> 13.1 mm
- net N$7: track 30.4 -> 15.1 mm
- net N$9: track 17.1 -> 3.07 mm
- net N$16: track 0.00 -> 13.8 mm
- net N$1: track 22.7 -> 9.96 mm
- net N$6: track 23.5 -> 12.0 mm
- net N$17: track 27.5 -> 36.9 mm
- net N$3: track 15.3 -> 9.45 mm
- net N$14: track 12.4 -> 6.91 mm
- net N$12: track 72.8 -> 78.1 mm
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Other:
- board text added: "+"
- board text added: "Delayed Start Unit v 0.1"
- board text added: "GND"
- board text added: "Vin"

Commit message: Nice routing
Parts:
- added LED6: (no value), led:LED3MM
- added R8: 350, eagle-ltspice:0204/7
- +: device SparkFun-Connectors:JST-2-PTH-VERT -> SparkFun-Connectors:1X02
- moved SW1 44.1 mm to (39.4, 12.7)
- moved SET_BTN 38.9 mm to (78.7, 33.0), turned to 90 degrees
- moved R6 34.5 mm to (87.6, 21.6), turned to 90 degrees
- moved + 32.0 mm to (33.0, 20.3), turned to 270 degrees
- moved VALID_BTN 27.1 mm to (67.3, 33.0), turned to 90 degrees
- moved R3 24.3 mm to (44.5, 29.2)
- moved R7 23.4 mm to (55.9, 29.2), turned to 90 degrees
- moved R4 23.3 mm to (40.6, 29.2)
- moved R1 20.1 mm to (52.1, 29.2), turned to 270 degrees
- moved R5 18.9 mm to (36.8, 29.2)
- moved R2 13.3 mm to (48.3, 29.2)
- moved LED2 12.7 mm to (57.1, 44.5)
- moved LED3 12.7 mm to (50.8, 44.5)
- moved LED1 12.7 mm to (63.5, 44.5)
- moved LED4 12.7 mm to (44.5, 44.5)
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Connections:
- removed net RELAY_1: ARDUINO_DUE.D4, RELAY.2
- new net N$18: ARDUINO_DUE.D13, LED6.A
- new net N$19: ARDUINO_DUE.D3, RELAY.3
- new net N$20: ARDUINO_DUE.D2, RELAY.2
- net GND: now also ARDUINO_DUE.GND@0, ARDUINO_DUE.GND@1, R8.2; no longer ARDUINO_DUE.GND@2
- net N$12: now also ARDUINO_DUE.D5, VALID_BTN.2; no longer ARDUINO_DUE.D2, SET_BTN.2
- net N$15: now also ARDUINO_DUE.D4, SET_BTN.2; no longer ARDUINO_DUE.D3, VALID_BTN.2
- net N$17: now also LED6.K, R8.1; no longer ARDUINO_DUE.D5, RELAY.3
Routing:
- net N$12: track 78.1 -> 27.7 mm
- net N$19: track 0.00 -> 30.8 mm
- net RELAY_1: track 29.2 -> 0.00 mm
- net GND: track 93.6 -> 120.5 mm
- net N$20: track 0.00 -> 26.0 mm
- net N$18: track 0.00 -> 25.1 mm
- net N$15: track 46.4 -> 25.3 mm
- net N$17: track 36.9 -> 18.3 mm
- net N$6: track 12.0 -> 28.2 mm
- net N$7: track 15.1 -> 31.2 mm
- net N$5: track 10.5 -> 26.0 mm
- net N$3: track 9.45 -> 23.5 mm
- net N$8: track 2.58 -> 14.6 mm
- net N$9: track 3.07 -> 13.5 mm
- net N$1: track 9.96 -> 19.7 mm
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Other:
- board text added: "github.com/xylome/arduino"
- board text removed: "+"
- board text removed: "GND"
- board text removed: "Vin"

Commit message: Reverse 4 PIN header for the relay
Parts:
- moved R6 6.35 mm to (81.3, 21.6)
- moved SET_BTN 3.81 mm to (74.9, 33.0)
- moved RELAY 2.84 mm to (85.1, 43.2), turned to 90 degrees
- moved VALID_BTN 2.54 mm to (64.8, 33.0)
Routing:
- net GND: track 120.5 -> 107.9 mm
- net N$19: track 30.8 -> 19.2 mm
- net N$13: track 65.7 -> 74.8 mm
- net N$11: track 15.5 -> 10.4 mm
- net N$14: track 11.8 -> 7.97 mm
- net N$5: track 26.0 -> 22.3 mm
- net N$6: track 28.2 -> 25.5 mm
- net N$20: track 26.0 -> 28.6 mm
- net VCC: track 30.4 -> 28.0 mm
- net N$3: track 23.5 -> 21.2 mm
- net N$7: track 31.2 -> 29.3 mm
- net N$12: track 27.7 -> 28.8 mm
- net N$18: track 25.1 -> 24.1 mm
- net N$2: track 18.7 -> 17.8 mm
